Commit message: fixed some j

File: src/depth_gazebo/urdf/robot_model.xacro (robot description, xacro)
@@ -48,6 +48,20 @@
         </visual>
     </link>
+ <link name="lidar_link">
+            <visual name='lidar_visual'>
+                <origin xyz="0 0 0" rpy=" 0 0 0"/>
+                <geometry>
+                    <box size=".05 .05 .05"/>
+                </geometry>
+                <material name="red"/>
+            </visual>
+        </link>
+ <joint name="lidar_joint" type="fixed">
+            <origin xyz="0.275 0 0.325" rpy="0 0 0"/>
+            <child link="lidar_link"/>
+            <parent link="base_link"/>
+ </joint>
   <!-- connecting depth camera  -->
-  <xacro:include filename="$(find realsense2_description)/urdf/test_d435_camera.urdf.xacro"/>
+  <!-- <xacro:include filename="$(find realsense2_description)/urdf/test_d435_camera.urdf.xacro"/> -->
   <xacro:wheel side="left" x="0.15" y="0.325" z="0.1"/>
   <xacro:wheel side="right" x="0.15" y="-0.325" z="0.1"/>
